Commit message: 增加gazebo fortress环境下的相机仿真

File: learning_gazebo/urdf/mbot_with_camera_gazebo.xacro (robot description, xacro)
@@ -1,4 +1,4 @@
 <?xml version="1.0"?>
-<robot name="arm" xmlns:xacro="http://www.ros.org/wiki/xacro">
+<robot name="mbot" xmlns:xacro="http://www.ros.org/wiki/xacro">
     <xacro:include filename="$(find learning_gazebo)/urdf/mbot_base_gazebo.xacro" />
     <xacro:include filename="$(find learning_gazebo)/urdf/sensors/camera_gazebo.xacro" />

File: learning_gazebo/urdf/mbot_with_kinect_gazebo.xacro (robot description, xacro)
@@ -1,4 +1,4 @@
 <?xml version="1.0"?>
-<robot name="arm" xmlns:xacro="http://www.ros.org/wiki/xacro">
+<robot name="mbot" xmlns:xacro="http://www.ros.org/wiki/xacro">
     <xacro:include filename="$(find learning_gazebo)/urdf/mbot_base_gazebo.xacro" />
     <xacro:include filename="$(find learning_gazebo)/urdf/sensors/kinect_gazebo.xacro" />

File: learning_gazebo/urdf/mbot_with_laser_gazebo.xacro (robot description, xacro)
@@ -1,4 +1,4 @@
 <?xml version="1.0"?>
-<robot name="arm" xmlns:xacro="http://www.ros.org/wiki/xacro">
+<robot name="mbot" xmlns:xacro="http://www.ros.org/wiki/xacro">
     <xacro:include filename="$(find learning_gazebo)/urdf/mbot_base_gazebo.xacro" />
     <xacro:include filename="$(find learning_gazebo)/urdf/sensors/lidar_gazebo.xacro" />

File: learning_gazebo/urdf/mbot_with_rgbd_gazebo.xacro (robot description, xacro)
@@ -1,4 +1,4 @@
 <?xml version="1.0"?>
-<robot name="arm" xmlns:xacro="http://www.ros.org/wiki/xacro">
+<robot name="mbot" xmlns:xacro="http://www.ros.org/wiki/xacro">
     <xacro:include filename="$(find learning_gazebo)/urdf/mbot_base_gazebo.xacro" />
     <xacro:include filename="$(find learning_gazebo)/urdf/sensors/rgbd_gazebo.xacro" />

File: learning_gazebo_fortress/urdf/mbot_base_gazebo_fortress.xacro (robot description, xacro)
@@ -166,11 +166,4 @@
                   <robot_base_frame>base_footprint</robot_base_frame>
             </plugin>
-			<plugin filename="ignition-gazebo-triggered-publisher-system"
-					name="ignition::gazebo::systems::TriggeredPublisher">
-				<input type="ignition.msgs.Empty" topic="/start"/>
-				<output type="ignition.msgs.Twist" topic="/cmd_vel">
-				linear: {x: 3}
-				</output>
-			</plugin>
         </gazebo>
     </xacro:macro>

File: learning_gazebo_fortress/urdf/mbot_with_camera_gazebo_fortress.xacro (robot description, xacro)
@@ -25,4 +25,15 @@
 	</gazebo>
     <xacro:include filename="$(find learning_gazebo_fortress)/urdf/mbot_base_gazebo_fortress.xacro" />
+    <xacro:include filename="$(find learning_gazebo_fortress)/urdf/sensors/camera_gazebo_fortress.xacro" />
+    <xacro:property name="camera_offset_x" value="0.17" />
+    <xacro:property name="camera_offset_y" value="0" />
+    <xacro:property name="camera_offset_z" value="0.10" />
+    <!-- Camera -->
+    <joint name="camera_joint" type="fixed">
+        <origin xyz="${camera_offset_x} ${camera_offset_y} ${camera_offset_z}" rpy="0 0 0" />
+        <parent link="base_link"/>
+        <child link="camera_link"/>
+    </joint>
+    <xacro:usb_camera prefix="camera"/>
     <xacro:mbot_base_gazebo/>
 </robot>
