Commit message: 优化gazebo fortress版本的接口配置文件

File: learning_gazebo_fortress/urdf/mbot_base_gazebo_fortress.xacro (robot description, xacro)
@@ -27,4 +27,5 @@
     <xacro:macro name="sphere_inertial_matrix" params="m r">
         <inertial>
+            <origin xyz="0 0 0" rpy="0 0 0"/>
             <mass value="${m}" />
             <inertia ixx="${2*m*r*r/5}" ixy="0" ixz="0"
@@ -35,4 +36,5 @@
     <xacro:macro name="cylinder_inertial_matrix" params="m r h">
         <inertial>
+            <origin xyz="0 0 0" rpy="0 0 0"/>
             <mass value="${m}" />
             <inertia ixx="${m*(3*r*r+h*h)/12}" ixy = "0" ixz = "0"
@@ -50,4 +52,10 @@
         </joint>
         <link name="${prefix}_wheel_link">
+            <collision>
+                <origin xyz="0 0 0" rpy="${M_PI/2} 0 0" />
+                <geometry>
+                    <cylinder radius="${wheel_radius}" length = "${wheel_length}"/>
+                </geometry>
+            </collision>
             <visual>
                 <origin xyz="0 0 0" rpy="${M_PI/2} 0 0" />
@@ -57,28 +65,10 @@
                 <material name="gray" />
             </visual>
-            <collision>
-                <origin xyz="0 0 0" rpy="${M_PI/2} 0 0" />
-                <geometry>
-                    <cylinder radius="${wheel_radius}" length = "${wheel_length}"/>
-                </geometry>
-            </collision>
             <xacro:cylinder_inertial_matrix  m="${wheel_mass}" r="${wheel_radius}" h="${wheel_length}" />
         </link>
         <gazebo reference="${prefix}_wheel_link">
-            <material>Gazebo/Gray</material>
             <mu1>100000.0</mu1>
             <mu2>100000.0</mu2>
         </gazebo>
-        <!-- Transmission is important to link the joints and the controller -->
-        <transmission name="${prefix}_wheel_joint_trans">
-            <type>transmission_interface/SimpleTransmission</type>
-            <joint name="${prefix}_wheel_joint" >
-                <hardwareInterface>hardware_interface/VelocityJointInterface</hardwareInterface>
-            </joint>
-            <actuator name="${prefix}_wheel_joint_motor">
-                <hardwareInterface>hardware_interface/VelocityJointInterface</hardwareInterface>
-                <mechanicalReduction>1</mechanicalReduction>
-            </actuator>
-        </transmission>
     </xacro:macro>
     <!-- Macro for robot caster -->
@@ -90,4 +80,10 @@
         </joint>
         <link name="${prefix}_caster_link">
+            <collision>
+                <origin xyz="0 0 0" rpy="0 0 0"/>
+                <geometry>
+                    <sphere radius="${caster_radius}" />
+                </geometry>
+            </collision>
             <visual>
                 <origin xyz="0 0 0" rpy="0 0 0"/>
@@ -97,34 +93,20 @@
                 <material name="black" />
             </visual>
-            <collision>
-                <origin xyz="0 0 0" rpy="0 0 0"/>
-                <geometry>
-                    <sphere radius="${caster_radius}" />
-                </geometry>
-            </collision>
             <xacro:sphere_inertial_matrix  m="${caster_mass}" r="${caster_radius}" />
         </link>
-        <gazebo reference="${prefix}_caster_link">
-            <material>Gazebo/Black</material>
-        </gazebo>
     </xacro:macro>
     <xacro:macro name="mbot_base_gazebo">
-        <link name="base_footprint">
-            <visual>
-                <origin xyz="0 0 0" rpy="0 0 0" />
-                <geometry>
-                    <box size="0.001 0.001 0.001" />
-                </geometry>
-            </visual>
-        </link>
-        <gazebo reference="base_footprint">
-            <turnGravityOff>false</turnGravityOff>
-        </gazebo>
+        <link name="base_footprint"/>
         <joint name="base_footprint_joint" type="fixed">
-            <origin xyz="0 0 ${base_length/2 + caster_radius*2}" rpy="0 0 0" />
             <parent link="base_footprint"/>
             <child link="base_link" />
         </joint>
         <link name="base_link">
+         	<collision>
+                <origin xyz=" 0 0 0" rpy="0 0 0" />
+                <geometry>
+                    <cylinder length="${base_length}" radius="${base_radius}"/>
+                </geometry>
+            </collision>
             <visual>
                 <origin xyz=" 0 0 0" rpy="0 0 0" />
@@ -134,15 +116,6 @@
                 <material name="yellow" />
             </visual>
-            <collision>
-                <origin xyz=" 0 0 0" rpy="0 0 0" />
-                <geometry>
-                    <cylinder length="${base_length}" radius="${base_radius}"/>
-                </geometry>
-            </collision>
             <xacro:cylinder_inertial_matrix  m="${base_mass}" r="${base_radius}" h="${base_length}" />
         </link>
-        <gazebo reference="base_link">
-            <material>Gazebo/Blue</material>
-        </gazebo>
         <xacro:wheel prefix="left"  reflect="1"/>
         <xacro:wheel prefix="right" reflect="-1"/>
@@ -166,4 +139,26 @@
                   <robot_base_frame>base_footprint</robot_base_frame>
             </plugin>
+            <plugin
+				filename="ignition-gazebo-sensors-system"
+				name="ignition::gazebo::systems::Sensors">
+				<render_engine>ogre</render_engine>
+			</plugin>
+			<plugin
+				filename="ignition-gazebo-user-commands-system"
+				name="ignition::gazebo::systems::UserCommands">
+			</plugin>
+			<plugin
+				filename="ignition-gazebo-scene-broadcaster-system"
+				name="ignition::gazebo::systems::SceneBroadcaster">
+			</plugin>
+			<plugin
+				filename="ignition-gazebo-joint-state-publisher-system"
+				name="ignition::gazebo::systems::JointStatePublisher"/>
+			<plugin
+				filename="ignition-gazebo-odometry-publisher-system"
+				name="ignition::gazebo::systems::OdometryPublisher">
+				<odom_frame>odom</odom_frame>
+				<robot_base_frame>base_footprint</robot_base_frame>
+			</plugin>
         </gazebo>
     </xacro:macro>

File: learning_gazebo_fortress/urdf/mbot_gazebo_fortress.xacro (robot description, xacro)
@@ -1,27 +1,4 @@
 <?xml version="1.0"?>
 <robot name="mbot" xmlns:xacro="http://www.ros.org/wiki/xacro">
-	<gazebo>
-		<physics name="1ms" type="ignored">
-		  <max_step_size>0.001</max_step_size>
-		  <real_time_factor>1.0</real_time_factor>
-		</physics>
-		<plugin
-		  filename="ignition-gazebo-physics-system"
-		  name="gz::sim::systems::Physics">
-		</plugin>
-		<plugin
-		  filename="ignition-gazebo-sensors-system"
-		  name="gz::sim::systems::Sensors">
-		  <render_engine>ogre</render_engine>
-		</plugin>
-		<plugin
-		  filename="ignition-gazebo-user-commands-system"
-		  name="gz::sim::systems::UserCommands">
-		</plugin>
-		<plugin
-		  filename="ignition-gazebo-scene-broadcaster-system"
-		  name="gz::sim::systems::SceneBroadcaster">
-		</plugin>
-	</gazebo>
     <xacro:include filename="$(find learning_gazebo_fortress)/urdf/mbot_base_gazebo_fortress.xacro" />
     <xacro:mbot_base_gazebo/>

File: learning_gazebo_fortress/urdf/mbot_with_camera_gazebo_fortress.xacro (robot description, xacro)
@@ -1,27 +1,4 @@
 <?xml version="1.0"?>
 <robot name="mbot" xmlns:xacro="http://www.ros.org/wiki/xacro">
-	<gazebo>
-		<physics name="1ms" type="ignored">
-		  <max_step_size>0.001</max_step_size>
-		  <real_time_factor>1.0</real_time_factor>
-		</physics>
-		<plugin
-		  filename="ignition-gazebo-physics-system"
-		  name="gz::sim::systems::Physics">
-		</plugin>
-		<plugin
-		  filename="ignition-gazebo-sensors-system"
-		  name="gz::sim::systems::Sensors">
-		  <render_engine>ogre</render_engine>
-		</plugin>
-		<plugin
-		  filename="ignition-gazebo-user-commands-system"
-		  name="gz::sim::systems::UserCommands">
-		</plugin>
-		<plugin
-		  filename="ignition-gazebo-scene-broadcaster-system"
-		  name="gz::sim::systems::SceneBroadcaster">
-		</plugin>
-	</gazebo>
     <xacro:include filename="$(find learning_gazebo_fortress)/urdf/mbot_base_gazebo_fortress.xacro" />
     <xacro:include filename="$(find learning_gazebo_fortress)/urdf/sensors/camera_gazebo_fortress.xacro" />

File: learning_gazebo_fortress/urdf/sensors/camera_gazebo_fortress.xacro (robot description, xacro)
@@ -25,7 +25,4 @@
             </collision>
         </link>
-        <gazebo reference="${prefix}_link">
-            <material>Gazebo/Black</material>
-        </gazebo>
         <gazebo reference="${prefix}_link">
             <sensor type="camera" name="camera_node">
